File: RPi_CM4_Sensor.kicad_pcb (KiCad board)
At the start: 2 copper layers, 48 x 72 mm, 16 parts, among them J1 RPi_pin, U1 SHT35, U2 SGP40, U3 APDS-9250, U4 SCD40

Commit message: fix: 微修正
Routing:
- net GND: vias 14 -> 40

Commit message: feat: 温度センサを別基板に配置するためのピンヘッダを追加
Parts:
- added J2: Conn_01x04_Male, Connector_PinHeader_2.54mm:PinHeader_1x04_P2.54mm_Vertical, F.Cu at (225.7, 54.1)
- moved C1 4.88 mm to (222.0, 62.1), turned to 180 degrees
- moved U1 4.52 mm to (218.7, 57.9)
Routing:
- net GND: track 38.6 -> 104.9 mm, vias 40 -> 27
- net PIN_05: track 149.2 -> 165.8 mm, vias 5 -> 6
- net PIN_03: track 141.0 -> 148.9 mm
- net +3V3: track 184.6 -> 185.9 mm
Other:
- outline, holes or cut-outs redrawn
- board text added: "APDS-9250"
- board text added: "ver 0.3 (2021.10.06)"
- board text removed: "ver 0.1 (2021.08.20)"
